File: Embedded/HUB75 Display Adapter/_autosave-HUB75 Display Adapter.kicad_sch (KiCad schematic)
At the start: 8 parts, among them J1 HUB75 Input, J2 Vertical, J3 JST [D], J4 JST [D], U1 Input A, U2 Input B

Commit message: Added Display Adapter for HUB75 Panels
Parts:
- J1: footprint Connector_PinHeader_2.54mm:PinHeader_2x08_P2.54mm_Vertical -> Connector_PinSocket_2.54mm:PinSocket_2x08_P2.54mm_Vertical
Changed lines of the file:
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@@
 			)
 		)
-		(property "Footprint" "Connector_PinHeader_2.54mm:PinHeader_2x08_P2.54mm_Vertical"
+		(property "Footprint" "Connector_PinSocket_2.54mm:PinSocket_2x08_P2.54mm_Vertical"
 			(at 64.77 85.09 0)
 			(effects
