File: Embedded/UI Display/UI Display.kicad_pcb (KiCad board)
At the start: 2 copper layers, 22.5 x 23.2 mm, 6 parts, among them J1 2.0 IPS Display, J2 SPI OLED, J3 5V-G I2C OLED, J4 G-5V I2C OLED, J5 SPI OLED, U2 FFC [U]

Commit message: Verified Combined Fabrication Files
Parts:
- added REF**: Logo_10mm, Logo:Logo_10mm, F.Cu at (155.0, 105.0)
Other:
- outline, holes or cut-outs redrawn
Changed lines of the file:
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@@
 		)
 		(fp_text user "${REFERENCE}"
-			(at 0 3.81 360)
+			(at 0 3.81 0)
 			(layer "F.Fab")
 			(effects
@@
 		)
 		(fp_text user "${REFERENCE}"
-			(at 0 7.62 360)
+			(at 0 7.62 0)
 			(layer "F.Fab")
 			(effects
@@
 		)
 		(fp_text user "${REFERENCE}"
-			(at 0 3.81 360)
+			(at 0 3.81 0)
 			(layer "F.Fab")
 			(effects
@@
 		)
 	)
+	(footprint "Logo:Logo_10mm"
+		(layer "F.Cu")
+		(at 155 105)
+		(property "Reference" "REF**"
+			(at 0 -3.5 0)
+			(unlocked yes)
+			(layer "F.SilkS")
+			(hide yes)
+			(effects
+				(font
+					(size 1 1)
+					(thickness 0.1)
+				)
+			)
+		)
+		(property "Value" "Logo_10mm"
+			(at 0 4.5 0)
+			(unlocked yes)
+			(layer "F.Fab")
+			(hide yes)
+			(effects
+				(font
+					(size 1 1)
+					(thickness 0.15)
+				)
+			)
+		)
+		(property "Footprint" "Logo:Logo_10mm"
+			(at 0 -3 0)
+			(unlocked yes)
+			(layer "F.Fab")
+			(hide yes)
+			(effects
+				(font
+					(size 1 1)
+					(thickness 0.15)
+				)
+			)
+		)
+		(property "Datasheet" ""
+			(at 0 -3 0)
+			(unlocked yes)
+			(layer "F.Fab")
+			(hide yes)
+			(effects
+				(font
+					(size 1 1)
+					(thickness 0.15)
+				)
+			)
+		)
+		(property "Description" ""
+			(at 0 -3 0)
+			(unlocked yes)
+			(layer "F.Fab")
+			(hide yes)
+			(effects
+				(font
+					(size 1 1)
+					(thickness 0.15)
+				)
+			)
+		)
+		(attr smd board_only)
+		(fp_poly
+			(pts
+				(xy 2.458919 -0.793871) (xy 2.496605 -0.748161) (xy 2.550117 -0.676888) (xy 2.616513 -0.584069)
+				(xy 2.692853 -0.47372) (xy 2.77 -0.359183) (xy 2.901293 -0.157235) (xy 3.0409 0.06598) (xy 3.186336 0.30594)
+				(xy 3.335122 0.558126) (xy 3.484774 0.818017) (xy 3.632811 1.081094) (xy 3.77675 1.342837) (xy 3.91411 1.598725)
+				(xy 4.042409 1.844239) (xy 4.159164 2.074859) (xy 4.261893 2.286064) (xy 4.348116 2.473334) (xy 4.415349 2.63215)
+				(xy 4.422381 2.65) (xy 4.465252 2.773183) (xy 4.501462 2.903019) (xy 4.530034 3.032749) (xy 4.54999 3.155613)
+				(xy 4.560353 3.26485) (xy 4.560146 3.353703) (xy 4.548393 3.41541) (xy 4.536 3.436) (xy 4.511305 3.452138)
+				(xy 4.477031 3.456951) (xy 4.428889 3.449041) (xy 4.362592 3.427009) (xy 4.273851 3.389457) (xy 4.158378 3.334985)
+				(xy 4.027969 3.270296) (xy 3.824633 3.170257) (xy 3.635459 3.082557) (xy 3.453928 3.004985) (xy 3.273523 2.935329)
+				(xy 3.087726 2.871378) (xy 2.89002 2.810921) (xy 2.673888 2.751747) (xy 2.432812 2.691645) (xy 2.160275 2.628404)
+				(xy 2.08848 2.612294) (xy 1.840251 2.558868) (xy 1.61876 2.515755) (xy 1.412658 2.48105) (xy 1.210594 2.452848)
+				(xy 1.00122 2.429243) (xy 0.99376 2.428491) (xy 0.913626 2.415171) (xy 0.871667 2.394948) (xy 0.86567 2.38593)
+				(xy 0.864807 2.362093) (xy 0.885295 2.338577) (xy 0.932598 2.311398) (xy 1.012181 2.27657) (xy 1.02 2.273377)
+				(xy 1.14007 2.215979) (xy 1.277388 2.136063) (xy 1.421708 2.040165) (xy 1.562784 1.934819) (xy 1.607363 1.898696)
+				(xy 1.827303 1.690843) (xy 2.019617 1.455881) (xy 2.182425 1.197315) (xy 2.313843 0.918651) (xy 2.411991 0.623396)
+				(xy 2.474985 0.315056) (xy 2.480824 0.271578) (xy 2.494666 0.089944) (xy 2.494589 -0.109198) (xy 2.48131 -0.308653)
+				(xy 2.455543 -0.491227) (xy 2.447424 -0.531344) (xy 2.424236 -0.648116) (xy 2.413287 -0.730494)
+				(xy 2.41448 -0.782139) (xy 2.427717 -0.806705) (xy 2.44 -0.81)
+			)
+			(stroke
+				(width 0)
+				(type solid)
+			)
+			(fill solid)
+			(layer "F.SilkS")
+		)
+		(fp_poly
+			(pts
+				(xy -0.139403 -2.232953) (xy 0.032295 -2.22827) (xy 0.182318 -2.218706) (xy 0.315213 -2.203888)
+				(xy 0.435524 -2.183442) (xy 0.547796 -2.156995) (xy 0.656577 -2.124171) (xy 0.747919 -2.091648)
+				(xy 0.99734 -1.976917) (xy 1.233928 -1.827758) (xy 1.453086 -1.648787) (xy 1.650212 -1.444619) (xy 1.820708 -1.219871)
+				(xy 1.959973 -0.979159) (xy 2.039491 -0.795424) (xy 2.099447 -0.612085) (xy 2.139291 -0.43304) (xy 2.161454 -0.244051)
+				(xy 2.168349 -0.04) (xy 2.166451 0.116135) (xy 2.158538 0.245706) (xy 2.142654 0.361944) (xy 2.116846 0.478075)
+				(xy 2.079159 0.607331) (xy 2.067243 0.644508) (xy 1.962289 0.905087) (xy 1.82336 1.15062) (xy 1.65417 1.377595)
+				(xy 1.458434 1.582499) (xy 1.239866 1.761819) (xy 1.002182 1.912043) (xy 0.749095 2.029658) (xy 0.527303 2.100689)
+				(xy 0.274014 2.152261) (xy 0.030962 2.173071) (xy -0.215919 2.164123) (xy -0.274289 2.158012) (xy -0.536665 2.111354)
+				(xy -0.787556 2.032895) (xy -1.03059 1.920843) (xy -1.269398 1.773403) (xy -1.507609 1.588785) (xy -1.61 1.498218)
+				(xy -1.898139 1.251635) (xy -2.184377 1.041438) (xy -2.466847 0.86896) (xy -2.562272 0.818857) (xy -2.634883 0.78343)
+				(xy -2.709843 0.749422) (xy -2.79285 0.714625) (xy -2.889604 0.676831) (xy -3.005803 0.633832) (xy -3.147145 0.58342)
+				(xy -3.319331 0.523385) (xy -3.37 0.505877) (xy -3.549492 0.441932) (xy -3.694324 0.385266) (xy -3.808645 0.333472)
+				(xy -3.896606 0.284141) (xy -3.962354 0.234864) (xy -4.01004 0.183235) (xy -4.043813 0.126843) (xy -4.051036 0.110607)
+				(xy -4.073402 0.033183) (xy -4.091216 -0.076021) (xy -4.092746 -0.091522) (xy -0.895984 -0.091522)
+				(xy -0.890091 0.087104) (xy -0.848531 0.26005) (xy -0.772024 0.421899) (xy -0.663833 0.564524) (xy -0.543447 0.672858)
+				(xy -0.406968 0.754072) (xy -0.284047 0.802668) (xy -0.172548 0.826446) (xy -0.040135 0.834675)
+				(xy 0.097454 0.827822) (xy 0.224482 0.806353) (xy 0.291881 0.78558) (xy 0.455426 0.701874) (xy 0.596097 0.587759)
+				(xy 0.709394 0.447635) (xy 0.783388 0.305041) (xy 0.805257 0.243687) (xy 0.819127 0.182952) (xy 0.826652 0.110857)
+				(xy 0.829488 0.01542) (xy 0.829681 -0.03) (xy 0.823257 -0.183417) (xy 0.801693 -0.309647) (xy 0.761551 -0.419758)
+				(xy 0.699392 -0.524814) (xy 0.659192 -0.578637) (xy 0.537105 -0.702107) (xy 0.392447 -0.796569)
+				(xy 0.231322 -0.860904) (xy 0.059831 -0.893994) (xy -0.115921 -0.894719) (xy -0.289832 -0.861962)
+				(xy -0.455798 -0.794602) (xy -0.471687 -0.78594) (xy -0.549158 -0.73129) (xy -0.633808 -0.653765)
+				(xy -0.713855 -0.565712) (xy -0.777516 -0.479476) (xy -0.797887 -0.444143) (xy -0.865489 -0.27041)
+				(xy -0.895984 -0.091522) (xy -4.092746 -0.091522) (xy -4.104347 -0.209028) (xy -4.112668 -0.357863)
+				(xy -4.11605 -0.514552) (xy -4.114364 -0.671118) (xy -4.107482 -0.819586) (xy -4.095274 -0.95198)
+				(xy -4.077612 -1.060326) (xy -4.070414 -1.09) (xy -4.00501 -1.258276) (xy -3.903292 -1.413537) (xy -3.764968 -1.555982)
+				(xy -3.589743 -1.685809) (xy -3.377325 -1.803218) (xy -3.127419 -1.908407) (xy -2.839733 -2.001575)
+				(xy -2.65 -2.051511) (xy -2.536677 -2.078167) (xy -2.428419 -2.10129) (xy -2.32094 -2.121283) (xy -2.209952 -2.138544)
+				(xy -2.091169 -2.153475) (xy -1.960302 -2.166475) (xy -1.813064 -2.177946) (xy -1.645169 -2.188287)
+				(xy -1.452328 -2.197899) (xy -1.230254 -2.207182) (xy -0.97466 -2.216536) (xy -0.83 -2.221464) (xy -0.566006 -2.229177)
+				(xy -0.337322 -2.233131)
+			)
+			(stroke
+				(width 0)
+				(type solid)
+			)
+			(fill solid)
+			(layer "F.SilkS")
+		)
+	)
 	(footprint "FFC_Connector:FFC Aliexpress 0.5mm 12P"
 		(layer "B.Cu")
@@
 		)
 	)
-	(gr_rect
-		(start 140 89.25)
-		(end 162.5 112.5)
+	(gr_line
+		(start 140 110)
+		(end 140 91.75)
 		(stroke
 			(width 0.05)
 			(type default)
 		)
-		(fill none)
 		(layer "Edge.Cuts")
 	)
+	(gr_line
+		(start 162.5 91.75)
+		(end 162.5 110)
+		(stroke
+			(width 0.05)
+			(type default)
+		)
+		(layer "Edge.Cuts")
+	)
+	(gr_line
+		(start 142.5 89.25)
+		(end 160 89.25)
+		(stroke
+			(width 0.05)
+			(type default)
+		)
+		(layer "Edge.Cuts")
+	)
+	(gr_arc
+		(start 162.5 110)
+		(mid 161.767767 111.767767)
+		(end 160 112.5)
+		(stroke
+			(width 0.05)
+			(type default)
+		)
+		(layer "Edge.Cuts")
+	)
+	(gr_line
+		(start 160 112.5)
+		(end 142.5 112.5)
+		(stroke
+			(width 0.05)
+			(type default)
+		)
+		(layer "Edge.Cuts")
+	)
+	(gr_arc
+		(start 142.5 112.5)
+		(mid 140.732233 111.767767)
+		(end 140 110)
+		(stroke
+			(width 0.05)
+			(type default)
+		)
+		(layer "Edge.Cuts")
+	)
+	(gr_arc
+		(start 160 89.25)
+		(mid 161.767767 89.982233)
+		(end 162.5 91.75)
+		(stroke
+			(width 0.05)
+			(type default)
+		)
+		(layer "Edge.Cuts")
+	)
+	(gr_arc
+		(start 140 91.75)
+		(mid 140.732233 89.982233)
+		(end 142.5 89.25)
+		(stroke
+			(width 0.05)
+			(type default)
+		)
+		(layer "Edge.Cuts")
+	)
