File: Embedded/Substructure Main/Substructure Snoot Board/Substructure Snoot Board.kicad_sch (KiCad schematic)
At the start: 2 parts, among them U1 D0, U2 D1

Commit message: Added 3V3 Reg & S Port
Parts:
- added BootSW1: SW_Push, Button-R-667843:Button-R-667843, symbol Switch:SW_Push
- added C1: 1uF, Capacitor_SMD:C_0603_1608Metric, symbol Device:C
- added C2: 22uF, Capacitor_SMD:C_0603_1608Metric_Pad1.08x0.95mm_HandSolder, symbol Device:C
- added C3: 0.1uF, Capacitor_SMD:C_0603_1608Metric_Pad1.08x0.95mm_HandSolder, symbol Device:C
- added ESP1: ESP32-S3-WROOM-1, PCM_Espressif:ESP32-S3-WROOM-1, symbol PCM_Espressif:ESP32-S3-WROOM-1
- added R1, R2: 10K, Resistor_SMD:R_0603_1608Metric, symbol Device:R
- added U4: S, FFC:FFC-8-0.5, symbol FFC:FFC-8
Connections:
- net +5V: now also U4.4, U4.5
- net GND: now also BootSW1.2, C1.1, C2.2, C3.2, ESP1.1 (GND), ESP1.40 (GND), ESP1.41 (GND), U4.1, U4.8
- new net: BootSW1.1, ESP1.27 (GPIO0/BOOT), R2.2
- new net: C1.2, ESP1.3 (EN), R1.2
- new net +3V3: C2.1, C3.1, ESP1.2 (3V3), R1.1, R2.1
- new net Main UART RX: U4.2
- new net Main UART TX: U4.3
- new net Main USB +: U4.6
- new net Main USB -: U4.7
- no-connect marks 0 -> 6
Other:
- added sheet 3V3 Reg (3V3 Reg.kicad_sch)
- moved on the sheet: U2
