File: Embedded/Substructure Snoot Board/Substructure Snoot Board.kicad_sch (KiCad schematic)
At the start: 37 parts, among them J1 10171746-00021LF, J2 PWR Jumper Pins, J3 L0 JST, J4 L1 JST, J5 5Vout, J6 A JST, J7 S Pins A, J8 S Pins B, J9 GNDout, U1 D0 FFC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

Commit message: Added All Signal Routing
Connections:
- net Addr LED 0: now also ESP1.17 (GPIO9/TOUCH9/ADC1_CH8/FSPIHD/SUBSPIHD); no longer ESP1.19 (GPIO11/TOUCH11/ADC2_CH0/FSPID/FSPIIO5/SUBSPID)
- net I2C SCL: now also ESP1.18 (GPIO10/TOUCH10/ADC1_CH9/FSPICS0/FSPIIO4/SUBSPICS0); no longer ESP1.17 (GPIO9/TOUCH9/ADC1_CH8/FSPIHD/SUBSPIHD)
- net I2C SDA: now also ESP1.19 (GPIO11/TOUCH11/ADC2_CH0/FSPID/FSPIIO5/SUBSPID); no longer ESP1.18 (GPIO10/TOUCH10/ADC1_CH9/FSPICS0/FSPIIO4/SUBSPICS0)
- net UI GPIO 0: now also ESP1.24 (GPIO47/SPICLK_P/SUBSPICLK_P_DIFF); no longer ESP1.21 (GPIO13/TOUCH13/ADC2_CH2/FSPIQ/FSPIIO7/SUBSPIQ)
- net UI GPIO 1: now also ESP1.23 (GPIO21); no longer ESP1.22 (GPIO14/TOUCH14/ADC2_CH3/FSPIWP/FSPIDQS/SUBSPIWP)
- net UI GPIO 2: now also ESP1.22 (GPIO14/TOUCH14/ADC2_CH3/FSPIWP/FSPIDQS/SUBSPIWP); no longer ESP1.23 (GPIO21)
- net UI GPIO 3: now also ESP1.21 (GPIO13/TOUCH13/ADC2_CH2/FSPIQ/FSPIIO7/SUBSPIQ); no longer ESP1.24 (GPIO47/SPICLK_P/SUBSPICLK_P_DIFF)
Changed lines of the file:
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@@
 (kicad_sch
-	(version 20231120)
+	(version 20250114)
 	(generator "eeschema")
-	(generator_version "8.0")
+	(generator_version "9.0")
 	(paper "A3")
 	(junction
@@
 	(global_label "UI GPIO 3"
 		(shape input)
-		(at 375.92 115.57 0)
+		(at 375.92 95.25 0)
 		(fields_autoplaced yes)
 		(effects
@@
 		)
 		(property "Intersheetrefs" "${INTERSHEET_REFS}"
-			(at 388.4605 115.57 0)
+			(at 388.4605 95.25 0)
 			(effects
 				(font
@@
 	(global_label "UI GPIO 0"
 		(shape input)
-		(at 375.92 95.25 0)
+		(at 375.92 115.57 0)
 		(fields_autoplaced yes)
 		(effects
@@
 		)
 		(property "Intersheetrefs" "${INTERSHEET_REFS}"
-			(at 388.4605 95.25 0)
+			(at 388.4605 115.57 0)
 			(effects
 				(font
@@
 	(global_label "I2C SDA"
 		(shape input)
-		(at 375.92 87.63 0)
+		(at 375.92 90.17 0)
 		(fields_autoplaced yes)
 		(effects
@@
 		)
 		(property "Intersheetrefs" "${INTERSHEET_REFS}"
-			(at 386.5252 87.63 0)
+			(at 386.5252 90.17 0)
 			(effects
 				(font
@@
 	(global_label "I2C SCL"
 		(shape input)
-		(at 375.92 85.09 0)
+		(at 375.92 87.63 0)
 		(fields_autoplaced yes)
 		(effects
@@
 		)
 		(property "Intersheetrefs" "${INTERSHEET_REFS}"
-			(at 386.4647 85.09 0)
+			(at 386.4647 87.63 0)
 			(effects
 				(font
@@
 	(global_label "UI GPIO 1"
 		(shape input)
-		(at 375.92 97.79 0)
+		(at 375.92 105.41 0)
 		(fields_autoplaced yes)
 		(effects
@@
 		)
 		(property "Intersheetrefs" "${INTERSHEET_REFS}"
-			(at 388.4605 97.79 0)
+			(at 388.4605 105.41 0)
 			(effects
 				(font
@@
 	(global_label "Addr LED 0"
 		(shape input)
-		(at 375.92 90.17 0)
+		(at 375.92 85.09 0)
 		(fields_autoplaced yes)
 		(effects
@@
 		)
 		(property "Intersheetrefs" "${INTERSHEET_REFS}"
-			(at 389.6698 90.17 0)
+			(at 389.6698 85.09 0)
 			(effects
 				(font
@@
 	(global_label "UI GPIO 2"
 		(shape input)
-		(at 375.92 105.41 0)
+		(at 375.92 97.79 0)
 		(fields_autoplaced yes)
 		(effects
@@
 		)
 		(property "Intersheetrefs" "${INTERSHEET_REFS}"
-			(at 388.4605 105.41 0)
+			(at 388.4605 97.79 0)
 			(effects
 				(font
@@
 		)
 	)
+	(embedded_fonts no)
 )
