File: Embedded/Substructure Boop Board/Substructure Boop Board.kicad_sch (KiCad schematic)
At the start: 41 parts, among them U1 PN5321A3HN_C1xx, U2 AD7142ACPZ-500RL7, U3 LD1117S33TR_SOT223, U4 0.35uH (Per Coil), U5 R FFC, Y1 7M-27.120MAAJ-T

Commit message: Added LCSC & Digikey IDs for main components
Parts:
- U1: LCSC (none) -> C28925
- U2: Digikey (none) -> 505-AD7142ACPZ-500RL7DKR-ND; LCSC (none) -> C208139
- U3: LCSC (none) -> C86781
- Y1: LCSC (none) -> C2450418
Changed lines of the file:
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@@
 			)
 		)
+		(property "LCSC" "C208139"
+			(at 203.2 25.4 0)
+			(effects
+				(font
+					(size 1.27 1.27)
+				)
+				(hide yes)
+			)
+		)
+		(property "Digikey" "505-AD7142ACPZ-500RL7DKR-ND"
+			(at 203.2 25.4 0)
+			(effects
+				(font
+					(size 1.27 1.27)
+				)
+				(hide yes)
+			)
+		)
 		(pin "8"
 		)
@@
 			)
 		)
+		(property "LCSC" "C2450418"
+			(at 46.99 175.26 0)
+			(effects
+				(font
+					(size 1.27 1.27)
+				)
+				(hide yes)
+			)
+		)
 		(pin "3"
 		)
@@
 			)
 		)
+		(property "LCSC" "C86781"
+			(at 93.98 30.48 0)
+			(effects
+				(font
+					(size 1.27 1.27)
+				)
+				(hide yes)
+			)
+		)
 		(pin "2"
 		)
@@
 			(at 99.06 143.51 0)
 			(effects
+				(font
+					(size 1.27 1.27)
+				)
+				(hide yes)
+			)
+		)
+		(property "LCSC" "C28925"
+			(at 99.06 143.51 0)
+			(effects

Commit message: Added LCSC IDs
Parts:
- C1: LCSC (none) -> C327025
- C10, C11, C16, C3, C4, C5, C6: LCSC (none) -> C1525
- C12, C13: LCSC (none) -> C70465
- C14: LCSC (none) -> C1591
- C15: LCSC (none) -> C3039698
- C17: LCSC (none) -> C14442
- C18, C23: LCSC (none) -> C86286
- C2, C7, C8, C9: LCSC (none) -> C15525
- C20, C25: LCSC (none) -> C307342
- C22, C26: LCSC (none) -> C307445
- L1, L2: LCSC (none) -> C502009
- R1, R2: LCSC (none) -> C163447
- R3: LCSC (none) -> C844716
- R4: LCSC (none) -> C482079
- R5, R6: LCSC (none) -> C482091
