File: Embedded/Substructure Main/RTC.kicad_sch (KiCad schematic)
At the start: 6 parts, among them U9 MCP7940N-xMNY, Y2 CM7V-T1A

Commit message: Modified Files (Synchronisation Update)
Parts:
- renumbered Coin_Cell to Coin_Cell1
Changed lines of the file:
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@@
 		(on_board yes)
 		(dnp no)
-		(property "Reference" "Coin_Cell"
+		(property "Reference" "Coin_Cell1"
 			(at 101.6 53.3401 0)
 			(effects
@@
 			(project "Substructure Main"
 				(path "/dda3f9ed-866a-496e-a4f2-d6745d13652e/cf64468b-2af6-4e81-8dd0-6dc57a236030"
-					(reference "Coin_Cell")
+					(reference "Coin_Cell1")
 					(unit 1)
 				)
