File: Embedded/Substructure Power Distribution/buckconverter.kicad_sch (KiCad schematic)
At the start: 43 parts, among them Q1 CSD17577Q5A, Q2 CSD17577Q5A, Q3 CSD17573Q5B, Q4 CSD17577Q5A, U1 LM5176PWP

Commit message: Added P Channel mosfets & crow bar circuits
Changed lines of the file:
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@@
 (kicad_sch
-	(version 20231120)
+	(version 20250114)
 	(generator "eeschema")
-	(generator_version "8.0")
+	(generator_version "9.0")
 	(paper "A2")
 	(junction

Commit message: Added Component Placement
Parts:
- removed C10, C21: 47uF 3mohm, Capacitor_SMD:C_1210_3225Metric_Pad1.33x2.70mm_HandSolder, symbol Device:C
- removed C3, C5, C6: 33uF 40mohm, Capacitors:EEFCX1E330R, symbol Device:C_Polarized
Other:
- moved on the sheet: C8
