File: Embedded/Substructure UI/Substructure UI.kicad_pcb (KiCad board)
At the start: 2 copper layers, 44 x 32 mm, 6 parts, among them J1 Conn_01x04_Socket, J2 Conn_01x04_Socket, U2 TLV74133PDBVR

Commit message: Modified Ports to fit FFC orientations
Connections:
- U1 pad 2: GPIO 0 -> GPIO 3
- U1 pad 3: GPIO 1 -> GPIO 2
- U1 pad 6: GPIO 2 -> GPIO 1
- U1 pad 7: GPIO 3 -> GPIO 0
Routing:
- net GPIO 0: track 28.8 -> 31.7 mm
- net GPIO 1: track 26.1 -> 28.3 mm
Changed lines of the file:
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@@
 			(size 0.3 1.1)
 			(layers "F.Cu" "F.Mask" "F.Paste")
-			(net 2 "GPIO 0")
+			(net 6 "GPIO 3")
 			(pintype "input")
 			(thermal_bridge_angle 45)
@@
 			(size 0.3 1.1)
 			(layers "F.Cu" "F.Mask" "F.Paste")
+			(net 7 "GPIO 2")
+			(pintype "input")
+			(thermal_bridge_angle 45)
+		)
+		(pad "4" smd rect
+			(at -0.25 -0.65)
+			(size 0.3 1.1)
+			(layers "F.Cu" "F.Mask" "F.Paste")
+			(net 5 "+5V")
+			(pintype "input")
+			(thermal_bridge_angle 45)
+		)
+		(pad "5" smd rect
+			(at 0.25 -0.65)
+			(size 0.3 1.1)
+			(layers "F.Cu" "F.Mask" "F.Paste")
+			(net 5 "+5V")
+			(pintype "input")
+			(thermal_bridge_angle 45)
+		)
+		(pad "6" smd rect
+			(at 0.750001 -0.65)
+			(size 0.3 1.1)
+			(layers "F.Cu" "F.Mask" "F.Paste")
 			(net 4 "GPIO 1")
 			(pintype "input")
 			(thermal_bridge_angle 45)
 		)
-		(pad "4" smd rect
-			(at -0.25 -0.65)
-			(size 0.3 1.1)
-			(layers "F.Cu" "F.Mask" "F.Paste")
-			(net 5 "+5V")
-			(pintype "input")
-			(thermal_bridge_angle 45)
-		)
-		(pad "5" smd rect
-			(at 0.25 -0.65)
-			(size 0.3 1.1)
-			(layers "F.Cu" "F.Mask" "F.Paste")
-			(net 5 "+5V")
-			(pintype "input")
-			(thermal_bridge_angle 45)
-		)
-		(pad "6" smd rect
-			(at 0.750001 -0.65)
-			(size 0.3 1.1)
-			(layers "F.Cu" "F.Mask" "F.Paste")
-			(net 7 "GPIO 2")
-			(pintype "input")
-			(thermal_bridge_angle 45)
-		)
 		(pad "7" smd rect
 			(at 1.25 -0.65)
 			(size 0.3 1.1)
 			(layers "F.Cu" "F.Mask" "F.Paste")
-			(net 6 "GPIO 3")
+			(net 2 "GPIO 0")
 			(pintype "input")
 			(thermal_bridge_angle 45)
@@
 	)
 	(segment
-		(start 95 65.3)
-		(end 92.57 65.3)
+		(start 104.3671 67.202)
+		(end 94.472 67.202)
 		(width 0.2)
 		(layer "F.Cu")
@@
 	)
 	(segment
-		(start 101.5349 64.5)
-		(end 95.8 64.5)
-		(width 0.2)
-		(layer "F.Cu")
-		(net 2)
-	)
-	(segment
-		(start 92.57 65.3)
+		(start 94.472 67.202)
 		(end 91.27 64)
 		(width 0.2)
@@
 	)
 	(segment
-		(start 102.25 65.95)
-		(end 102.25 65.2151)
+		(start 104.75 65.95)
+		(end 104.75 66.8191)
 		(width 0.2)
 		(layer "F.Cu")
@@
 	)
 	(segment
-		(start 102.25 65.2151)
-		(end 101.5349 64.5)
+		(start 104.75 66.8191)
+		(end 104.3671 67.202)
 		(width 0.2)
 		(layer "F.Cu")
@@
 	)
 	(segment
-		(start 95.8 64.5)
-		(end 95 65.3)
-		(width 0.2)
-		(layer "F.Cu")
-		(net 2)
-	)
-	(segment
-		(start 101.602 64)
-		(end 102.75 65.148)
-		(width 0.2)
-		(layer "F.Cu")
-		(net 4)
-	)
-	(segment
-		(start 102.75 65.148)
-		(end 102.75 65.950001)
+		(start 93.81 64)
+		(end 96.611 66.801)
 		(width 0.2)
 		(layer "F.Cu")
@@
 	)
 	(segment
-		(start 93.81 64)
-		(end 101.602 64)
+		(start 96.611 66.801)
+		(end 104.201 66.801)
 		(width 0.2)
 		(layer "F.Cu")
+		(net 4)
+	)
+	(segment
+		(start 104.201 66.801)
+		(end 104.250001 66.751999)
+		(width 0.2)
+		(layer "F.Cu")
+		(net 4)
+	)
+	(segment
+		(start 104.250001 66.751999)
+		(end 104.250001 65.95)
+		(width 0.2)
+		(layer "F.Cu")

Commit message: Added Logos
Parts:
- added G***: LOGO, LOGO, B.Cu at (90.5, 57.5)
Changed lines of the file:
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@@
 		)
+	)
+	(footprint "LOGO"
+		(layer "B.Cu")
+		(at 90.5 57.5 180)
+		(property "Reference" "G***"
+			(at 0 0 0)
+			(layer "B.SilkS")
+			(hide yes)
+			(effects
+				(font
+					(size 1.5 1.5)
+					(thickness 0.3)
+				)
+				(justify mirror)
+			)
+		)
+		(property "Value" "LOGO"
+			(at 0.75 0 0)
+			(layer "B.SilkS")
+			(hide yes)
+			(effects
+				(font
+					(size 1.5 1.5)
+					(thickness 0.3)
+				)
+				(justify mirror)
+			)
+		)
+		(property "Datasheet" ""
+			(at 0 0 0)
+			(layer "B.Fab")
+			(hide yes)
+			(effects
+				(font
+					(size 1.27 1.27)
+					(thickness 0.15)
+				)
+				(justify mirror)
+			)
+		)
+		(property "Description" ""
+			(at 0 0 0)
+			(layer "B.Fab")
+			(hide yes)
+			(effects
+				(font
+					(size 1.27 1.27)
+					(thickness 0.15)
+				)
+				(justify mirror)
+			)
+		)
+		(attr board_only exclude_from_pos_files exclude_from_bom)
+		(fp_poly
+			(pts
+				(xy 3.446033 2.099779) (xy 3.638973 1.850672) (xy 3.891791 1.483316) (xy 4.179959 1.036896) (xy 4.478949 0.550595)
+				(xy 4.764234 0.063598) (xy 5.011285 -0.38491) (xy 5.195574 -0.755744) (xy 5.227026 -0.827154) (xy 5.448479 -1.399299)
+				(xy 5.654597 -2.024482) (xy 5.828353 -2.641096) (xy 5.952723 -3.187536) (xy 6.010683 -3.602197)
+				(xy 6.012831 -3.670632) (xy 5.974358 -3.891591) (xy 5.844609 -3.9734) (xy 5.60209 -3.913169) (xy 5.225305 -3.708007)
+				(xy 4.945132 -3.527052) (xy 4.163679 -3.047051) (xy 3.426405 -2.675299) (xy 2.775134 -2.431127)
+				(xy 2.390234 -2.346125) (xy 1.951324 -2.258473) (xy 1.730006 -2.128862) (xy 1.720289 -1.938477)
+				(xy 1.916179 -1.668501) (xy 2.113106 -1.475854) (xy 2.678363 -0.827611) (xy 3.048417 -0.090821)
+				(xy 3.232627 0.756914) (xy 3.258117 1.264239) (xy 3.267399 1.688916) (xy 3.291092 2.011293) (xy 3.324711 2.178983)
+				(xy 3.337499 2.191451)
+			)
+			(stroke
+				(width 0)
+				(type solid)
+			)
+			(fill yes)
+			(layer "B.SilkS")
+		)
+		(fp_poly
+			(pts
+				(xy -0.120747 4.190799) (xy 0.436967 4.139555) (xy 0.881297 4.04249) (xy 1.249124 3.890439) (xy 1.577332 3.674233)
+				(xy 1.902803 3.384705) (xy 2.026972 3.260178) (xy 2.443599 2.765161) (xy 2.703672 2.264802) (xy 2.834927 1.686996)
+				(xy 2.865929 1.079148) (xy 2.811482 0.408737) (xy 2.627809 -0.14326) (xy 2.284407 -0.660365) (xy 2.190237 -0.771097)
+				(xy 1.6066 -1.308885) (xy 0.959787 -1.644763) (xy 0.204354 -1.800509) (xy 0.016216 -1.81289) (xy -0.429975 -1.817888)
+				(xy -0.823051 -1.796616) (xy -1.074263 -1.754532) (xy -1.45649 -1.602926) (xy -1.828733 -1.388269)
+				(xy -2.255106 -1.070385) (xy -2.528762 -0.843076) (xy -3.053397 -0.420406) (xy -3.525978 -0.10504)
+				(xy -4.030201 0.150246) (xy -4.649759 0.392672) (xy -4.832744 0.456896) (xy -5.26317 0.612345) (xy -5.619 0.753126)
+				(xy -5.840229 0.855091) (xy -5.872346 0.875234) (xy -5.987886 1.093921) (xy -5.990275 1.168403)
+				(xy -1.17759 1.168403) (xy -1.085663 0.730785) (xy -0.837781 0.402654) (xy -0.484772 0.205371) (xy -0.077465 0.160299)
+				(xy 0.333311 0.288803) (xy 0.545535 0.444192) (xy 0.792785 0.808283) (xy 0.860943 1.227327) (xy 0.760982 1.638045)
+				(xy 0.503875 1.977159) (xy 0.252973 2.131207) (xy -0.205392 2.219145) (xy -0.621583 2.113164) (xy -0.949791 1.844094)
+				(xy -1.144207 1.442766) (xy -1.17759 1.168403) (xy -5.990275 1.168403) (xy -5.99933 1.450709) (xy -5.920399 1.892276)
+				(xy -5.764816 2.365296) (xy -5.546303 2.816445) (xy -5.278584 3.1924) (xy -5.275019 3.196359) (xy -4.935632 3.497303)
+				(xy -4.510664 3.777799) (xy -4.297955 3.885764) (xy -4.059775 3.981861) (xy -3.817157 4.052968)
+				(xy -3.528586 4.104033) (xy -3.152544 4.140003) (xy -2.647513 4.165825) (xy -1.971976 4.186446)
+				(xy -1.723856 4.1925) (xy -0.828727 4.205392)
+			)
+			(stroke
+				(width 0)
+				(type solid)
+			)
+			(fill yes)
+			(layer "B.SilkS")
+		)
+		(embedded_fonts no)
 	)
 	(gr_circle
