File: Embedded/Substructure Display Adapter/_autosave-Substructure Display Adapter.kicad_pcb (KiCad board)
At the start: 2 copper layers, 29 x 70 mm, 18 parts, among them J1 HUB75, J2 Input, J3 Output, J4 HUB75, J5 Input, J6 Output, U1 D0 FFC, U2 74HC245D_653, U3 74HC245D_653, U4 D0 FFC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

Commit message: Added Routing for right adapter
Parts:
- C3, C4, U5, U6: moved to B.Cu
- J4, J5, J6, JP2, U4: moved to F.Cu
- moved JP2 26.0 mm to (115.0, 93.0)
- moved C4 25.0 mm to (108.0, 68.0), turned to -90 degrees
- moved J5 23.8 mm to (116.0, 68.2), turned to -90 degrees
- moved J4 17.8 mm to (125.3, 88.9)
- moved U6 15.0 mm to (115.0, 73.0)
- moved U4 14.0 mm to (112.0, 87.0), turned to -90 degrees
- moved U5 13.0 mm to (115.0, 87.0)
- moved J6 11.9 mm to (132.0, 86.0), turned to 90 degrees
- moved C3 3.16 mm to (108.0, 82.0), turned to -90 degrees
- moved J2 0.25 mm to (116.4, 44.2)
Connections:
- U6 pad 11: unconnected-(U6-B7-Pad11) -> Alt Disp GPIO 14
- U6 pad 12: unconnected-(U6-B6-Pad12) -> Alt Disp GPIO 13
- U6 pad 13: Alt Disp GPIO 14 -> Alt Disp GPIO 12
- U6 pad 14: Alt Disp GPIO 13 -> Alt Disp GPIO 11
- U6 pad 15: Alt Disp GPIO 12 -> Alt Disp GPIO 10
- U6 pad 16: Alt Disp GPIO 11 -> Alt Disp GPIO 9
- U6 pad 17: Alt Disp GPIO 10 -> unconnected-(U6-B1-Pad17)
- U6 pad 18: Alt Disp GPIO 9 -> unconnected-(U6-B0-Pad18)
Routing:
- net +5V: track 0.00 -> 55.9 mm, vias 0 -> 2
- net OE: track 0.00 -> 28.6 mm
- net Disp GPIO 9: track 0.00 -> 20.1 mm, vias 0 -> 1
- net GND: track 0.00 -> 20.0 mm, vias 0 -> 9
- net Disp GPIO 10: track 0.00 -> 17.9 mm, vias 0 -> 1
- net Disp GPIO 11: track 0.00 -> 15.8 mm, vias 0 -> 1
- net Disp GPIO 12: track 0.00 -> 13.7 mm, vias 0 -> 1
- net Disp GPIO 13: track 0.00 -> 11.5 mm, vias 0 -> 1
- net Disp Display Select: track 0.00 -> 10.6 mm, vias 0 -> 1
- net Disp GPIO 5: track 0.00 -> 10.1 mm, vias 0 -> 1
- net Disp GPIO 4: track 0.00 -> 9.41 mm, vias 0 -> 1
- net Disp GPIO 14: track 0.00 -> 9.36 mm, vias 0 -> 1
- net Disp GPIO 6: track 0.00 -> 9.34 mm, vias 0 -> 1
- net Disp GPIO 3: track 0.00 -> 8.64 mm, vias 0 -> 1
- net Disp GPIO 8: track 0.00 -> 8.48 mm
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