File: Embedded/Main Head CPU/Main Head CPU.kicad_sch (KiCad schematic)
At the start: 46 parts, among them J1 10171746-00021LF, J10 Extra, J11 Conn_01x06, J12 Substructure Port, J13 Conn_01x02_Socket, J2 Fan 0, J3 Fan 1, J4 MicroSD, J5 Maw, J6 Tongue, J7 Left Fin, J8 Right Fin, J9 Scales, Q1 DMG3402L, Q2 DMG3402L, U11 Sensored, U5 Buttons, U6 LD1117S33TR_SOT223, U7 LD1117S50TR_SOT223

Commit message: Added Footprints to components
Parts:
- J11: footprint (none) -> Connector_PinHeader_2.54mm:PinHeader_1x06_P2.54mm_Vertical
- U5: footprint FFC:FFC-8-0.5 -> FCC:FFC 0.8mm 8P
Changed lines of the file:
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@@
 		(dnp no)
 		(fields_autoplaced yes)
-		(property "Reference" "#PWR010"
+		(property "Reference" "#PWR0101"
 			(at 148.59 228.6 0)
 			(effects
@@
 			(project "Main Head CPU"
 				(path "/f158cce9-f45f-474d-a65f-ecbb8fa57101"
-					(reference "#PWR010")
+					(reference "#PWR0101")
 					(unit 1)
 				)
@@
 			)
 		)
-		(property "Footprint" "FFC:FFC-8-0.5"
+		(property "Footprint" "FCC:FFC 0.8mm 8P"
 			(at 101.6 172.72 0)
 			(effects
@@
 			)
 		)
-		(property "Footprint" ""
+		(property "Footprint" "Connector_PinHeader_2.54mm:PinHeader_1x06_P2.54mm_Vertical"
 			(at 102.87 261.62 0)
 			(effects

Commit message: Added Component placement positions
Parts:
- removed JP2, JP3: SolderJumper_3_Open, Jumper:SolderJumper-3_P1.3mm_Open_RoundedPad1.0x1.5mm, symbol Jumper:SolderJumper_3_Open
- added D3: PMEG3050EP_115, PMEG Diode:DIO_PMEG3050EP_115, symbol PMEG Diode:PMEG3050EP_115
- added SW2: RST, Buttons:R-667843, symbol Switch:SW_Push
- R7, R8: footprint Resistor_SMD:R_0402_1005Metric_Pad0.72x0.64mm_HandSolder -> Capacitor_SMD:C_0603_1608Metric_Pad1.08x0.95mm_HandSolder
- SW1: renamed from BootSW1; value SW_Push -> Boot
- renumbered C5 to C1, C9 to C10, C1 to C2, C2 to C3, C3 to C4, C4 to C5, C8 to C7, C10 to C8, C7 to C9, J3 to J10, J12 to J11, J13 to J12, J4 to J13, J5 to J2, J6 to J3, J7 to J4, J8 to J5, J9 to J6, J10 to J7, J11 to J8, J2 to J9, R5 to R1, R4 to R10, R6 to R2, R1 to R3, R9 to R4, R2 to R5, R10 to R6, R3 to R9, U11 to U1, U5 to U2, U6 to U3, U7 to U4
Connections:
- net +5RAW is gone; now on net +RAWVS: C2.1, C3.1, U3.3 (VI), U4.3 (VI)
- net +5V: now also J10.1 (Pin_1), J9.1 (Pin_1)
- net +RAWVS: now also D3.K
- net GND: now also SW2.2
- net at C6.2, ESP1.3 (EN), R9.2: now also SW2.1
- net +5VUSB: no longer names the net of C1.1, J1.A4_B9 (VBUS_A), J1.B4_A9 (VBUS_B)
- net +5VUSB: now also D3.A
Other:
- moved on the sheet: C6
