File: Embedded/Recondensed/Main Head CPU/Main Head CPU.kicad_pcb (KiCad board)
At the start: 4 copper layers, 50 x 47.5 mm, 53 parts, among them J1 10171746-00021LF, J10 Fan 1, J11 Substructure Power, J12 Head Power, J13 MicroSD, J14 Mic, J15 Expansion, J2 LEDs 0, J3 LEDs 1, J4 LEDs 2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

Commit message: Added LCSC Component IDs
Parts:
- removed SW1: Boot, Buttons:R-667843
- removed SW2: RST, Buttons:R-667843
- added S1: Boot, Buttons:SW_B3U-1000P, F.Cu at (109.5, 45.2)
- added S2: RST, Buttons:SW_B3U-1000P, F.Cu at (90.5, 45.2)
- J1: footprint USBC:AMPHENOL_10171746-00021LF -> USBC:MOLEX_2171790001
- R7: value 155ohm min -> 145ohm
- R8: value 70ohm min -> 33ohm
- moved J1 1.15 mm to (100.0, 86.9)
Routing:
- net GND: track 37.4 -> 38.8 mm

Commit message: Updated Asset Dates
Other:
- board text added: "Des: CSF-Main-CPU M/N: CSF-AAA-001 Rev: D0.0 Dat: 27.07.2025"
- board text removed: "Des: CSF-Main-CPU M/N: CSF-AAA-001 Rev: D0.0 Dat: 26.07.2025"
Changed lines of the file:
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@@
 		(layer "Edge.Cuts")
 	)
-	(gr_text "Des: CSF-Main-CPU\nM/N: CSF-AAA-001\nRev: D0.0\nDat: 26.07.2025"
+	(gr_text "Des: CSF-Main-CPU\nM/N: CSF-AAA-001\nRev: D0.0\nDat: 27.07.2025"
 		(at 104 72 0)
 		(layer "B.SilkS")

Commit message: Added Pullups for MicroSD & Modified Silkscreen
Parts:
- added R15: 10K, Resistor_SMD:R_0603_1608Metric_Pad0.98x0.95mm_HandSolder, F.Cu at (116.6, 83.8)
- added R16: 10K, Resistor_SMD:R_0603_1608Metric_Pad0.98x0.95mm_HandSolder, F.Cu at (113.3, 83.8)
- added R17: 10K, Resistor_SMD:R_0603_1608Metric_Pad0.98x0.95mm_HandSolder, F.Cu at (110.1, 83.8)
- added R18: 10K, Resistor_SMD:R_0603_1608Metric_Pad0.98x0.95mm_HandSolder, F.Cu at (109.1, 85.3)
- added R19: 10K, Resistor_SMD:R_0603_1608Metric_Pad0.98x0.95mm_HandSolder, F.Cu at (106.8, 83.8)
- added R20: 10K, Resistor_SMD:R_0603_1608Metric_Pad0.98x0.95mm_HandSolder, F.Cu at (115.5, 85.3)
Connections:
- J13 pad 1: unconnected-(J13-Pad1) -> Net-(J13-Pad1)
- J13 pad 8: unconnected-(J13-Pad8) -> Net-(J13-Pad8)
Routing:
- net SD SPI MISO: track 11.9 -> 19.1 mm
- net Net-(J13-Pad1): track 0.00 -> 7.08 mm
- net Net-(J13-Pad8): track 0.00 -> 5.81 mm
- net SD SPI CLK: track 13.3 -> 19.0 mm
- net SD SPI CS: track 15.3 -> 20.8 mm
- net SD SPI MOSI: track 15.5 -> 20.9 mm
- net +3V3: track 6.09 -> 8.00 mm
Other:
- board text added: "Des: CSF-Main-CPU M/N: CSF-AAA-001 Rev: D0.0 Dat: 28.07.2025"
- board text removed: "Des: CSF-Main-CPU M/N: CSF-AAA-001 Rev: D0.0 Dat: 27.07.2025"
